File: Schematic/Linear regulator STD/Linear regulator STD.kicad_pcb (KiCad board)
At the start: 2 copper layers, 15.2 x 37.3 mm, 13 parts, among them J1 Screw_Terminal_01x04, U1 LM317T

Commit message: PCB routing
Parts:
- moved D2 0.13 mm to (133.9, 88.8)
- moved J1 0.06 mm to (136.0, 95.8)
Routing:
- net /VIN: track 15.0 -> 30.9 mm
- net GND: track 7.02 -> 15.9 mm, vias 0 -> 3
- net Net-(C4-Pad1): track 14.4 -> 21.4 mm
Changed lines of the file:
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@@
-(kicad_pcb (version 20171130) (host pcbnew "(5.1.0)-1")
+(kicad_pcb (version 20171130) (host pcbnew 5.1.2-f72e74a~84~ubuntu19.04.1)
   (general
     (thickness 1.6)
     (drawings 12)
-    (tracks 45)
+    (tracks 72)
     (zones 0)
     (modules 13)
@@
   )
   (setup
-    (last_trace_width 0.3048)
+    (last_trace_width 0.4572)
     (user_trace_width 0.3048)
     (user_trace_width 0.4572)
@@
   )
   (module Connector_PinHeader_2.54mm_OSHW:PinHeader_1x04_P2.54mm_Horizontal (layer F.Cu)
-    (at 135.89 95.758 90)
+    (at 135.9535 95.758 90)
     (descr "Through hole angled pin header, 1x04, 2.54mm pitch, 6mm pin length, single row")
     (tags "Through hole angled pin header THT 1x04 2.54mm single row")
@@
   )
   (module Diode_SMD:D_SOD-123F (layer F.Cu)
-    (at 133.858 88.646 90)
+    (at 133.858 88.773 90)
     (descr D_SOD-123F)
     (tags D_SOD-123F)
@@
   (segment (start 145.2512 83.933) (end 144.6783 84.5059) (width 0.3048) (layer F.Cu) (net 1))
   (segment (start 138.176 89.001) (end 142.24 89.001) (width 0.8) (layer F.Cu) (net 1))
+  (via (at 135.382 85.852) (size 0.8) (drill 0.4) (layers F.Cu B.Cu) (net 1))
+  (segment (start 134.1485 85.852) (end 133.858 85.5615) (width 0.3048) (layer F.Cu) (net 1))
+  (segment (start 135.382 85.852) (end 134.1485 85.852) (width 0.3048) (layer F.Cu) (net 1))
+  (via (at 140.97 90.17) (size 0.8) (drill 0.4) (layers F.Cu B.Cu) (net 1))
+  (via (at 144.526 87.122) (size 0.8) (drill 0.4) (layers F.Cu B.Cu) (net 1))
+  (segment (start 144.6783 86.9697) (end 144.526 87.122) (width 0.3048) (layer F.Cu) (net 1))
+  (segment (start 144.6783 85.852) (end 144.6783 86.9697) (width 0.3048) (layer F.Cu) (net 1))
+  (segment (start 142.139 89.001) (end 140.97 90.17) (width 0.3048) (layer F.Cu) (net 1))
+  (segment (start 142.24 89.001) (end 142.139 89.001) (width 0.3048) (layer F.Cu) (net 1))
+  (segment (start 140.321 91.948) (end 140.321 93.1405) (width 0.4572) (layer F.Cu) (net 1))
+  (segment (start 141.0335 93.853) (end 141.0335 95.758) (width 0.4572) (layer F.Cu) (net 1))
+  (segment (start 140.321 93.1405) (end 141.0335 93.853) (width 0.4572) (layer F.Cu) (net 1))
   (segment (start 142.364 91.694) (end 142.364 92.7578) (width 0.4572) (layer F.Cu) (net 2))
-  (segment (start 143.51 93.9038) (end 143.51 95.758) (width 0.4572) (layer F.Cu) (net 2))
   (segment (start 142.364 92.7578) (end 143.51 93.9038) (width 0.4572) (layer F.Cu) (net 2))
   (segment (start 145.3642 93.9038) (end 143.51 93.9038) (width 0.3048) (layer F.Cu) (net 2))
@@
   (segment (start 135.514072 91.448928) (end 135.514072 90.84041) (width 0.3048) (layer F.Cu) (net 2))
   (segment (start 135.015 91.948) (end 135.514072 91.448928) (width 0.3048) (layer F.Cu) (net 2))
+  (segment (start 143.51 94.492419) (end 143.51 93.9038) (width 0.4572) (layer F.Cu) (net 2))
+  (segment (start 143.5735 94.555919) (end 143.51 94.492419) (width 0.4572) (layer F.Cu) (net 2))
+  (segment (start 143.5735 95.758) (end 143.5735 94.555919) (width 0.4572) (layer F.Cu) (net 2))
   (segment (start 133.858 88.1008) (end 133.858 87.246) (width 0.3048) (layer F.Cu) (net 3))
   (segment (start 132.955599 89.003201) (end 133.858 88.1008) (width 0.3048) (layer F.Cu) (net 3))
@@
   (segment (start 133.858 82.5865) (end 135.7862 82.5865) (width 0.3048) (layer F.Cu) (net 3))
   (segment (start 135.7862 82.5865) (end 135.9427 82.43) (width 0.3048) (layer F.Cu) (net 3))
+  (segment (start 134.23694 87.122) (end 134.11294 87.246) (width 0.3048) (layer F.Cu) (net 3))
+  (segment (start 137.2 84.2428) (end 136.144 85.2988) (width 0.3048) (layer F.Cu) (net 3))
+  (segment (start 137.2 82.43) (end 137.2 84.2428) (width 0.3048) (layer F.Cu) (net 3))
+  (segment (start 134.11294 87.246) (end 133.858 87.246) (width 0.3048) (layer F.Cu) (net 3))
+  (segment (start 136.144 85.2988) (end 136.144 86.36) (width 0.3048) (layer F.Cu) (net 3))
+  (segment (start 135.382 87.122) (end 134.23694 87.122) (width 0.3048) (layer F.Cu) (net 3))
+  (segment (start 136.144 86.36) (end 135.382 87.122) (width 0.3048) (layer F.Cu) (net 3))
   (segment (start 142.28 85.711) (end 142.24 85.751) (width 0.8) (layer F.Cu) (net 4))
   (segment (start 142.28 82.43) (end 142.28 85.711) (width 0.8) (layer F.Cu) (net 4))
@@
   (segment (start 144.5374 82.183) (end 146.05 82.183) (width 0.3048) (layer F.Cu) (net 4))
   (segment (start 144.2904 82.43) (end 144.5374 82.183) (width 0.3048) (layer F.Cu) (net 4))
+  (segment (start 142.28 82.4775) (end 142.24 82.5175) (width 0.4572) (layer B.Cu) (net 4))
+  (segment (start 142.28 82.43) (end 142.28 82.4775) (width 0.4572) (layer B.Cu) (net 4))
+  (segment (start 142.24 82.5175) (end 142.24 84.582) (width 0.4572) (layer B.Cu) (net 4))
+  (segment (start 142.24 84.582) (end 142.24 85.979) (width 0.4572) (layer B.Cu) (net 4))
+  (segment (start 135.9535 92.2655) (end 135.9535 95.758) (width 0.4572) (layer B.Cu) (net 4))
+  (segment (start 142.24 85.979) (end 135.9535 92.2655) (width 0.4572) (layer B.Cu) (net 4))
   (segment (start 146.2533 87.6947) (end 146.2532 87.6948) (width 0.3048) (layer F.Cu) (net 5))
   (segment (start 146.2533 85.852) (end 146.2533 87.6947) (width 0.3048) (layer F.Cu) (net 5))
